File: hardware/pcb/BLK_SWITCH_LED.kicad_sch (KiCad schematic)
At the start: 8 parts, among them J14 IDC-10_SWITCH_LED_DATA, J15 IDC-6_ZONE_INFO_12V, U12 74AHCT125, U13 ULN2803A

Commit message: Update hardware schematics and documentation; added source of truth for hardware, removed unused symbols, and modified connector specifications.
Parts:
- C51: symbol Device:C_Polarized -> Device:C_Small
- J15: value IDC-6_ZONE_INFO_12V -> IDC-10_ZONE_INFO_12V; footprint Connector_IDC:IDC-Header_2x03_P2.54mm_Vertical -> Connector_IDC:IDC-Header_2x05_P2.54mm_Vertical; symbol Connector_Generic:Conn_02x03_Odd_Even -> Connector_Generic:Conn_02x05_Odd_Even
Connections:
- net GNDPWR: now also J15.8 (Pin_8)
- no-connect marks 13 -> 16
Changed lines of the file:
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@@
-	)
-	(junction
-		(at 257.81 147.32)
-		(diameter 0)
-		(color 0 0 0 0)
 	)
 	(junction
@@
 	)
 	(no_connect
+		(at 133.35 66.04)
+	)
+	(no_connect
 		(at 194.31 39.37)
 	)
@@
 	)
 	(no_connect
+		(at 133.35 71.12)
+	)
+	(no_connect
 		(at 173.99 49.53)
 	)
@@
 		(at 194.31 46.99)
 	)
+	(no_connect
+		(at 146.05 71.12)
+	)
 	(wire
 		(pts
@@
 	(wire
 		(pts
-			(xy 184.15 147.32) (xy 257.81 147.32)
-		)
-		(stroke
-			(width 0)
-			(type default)
-		)
-	)
-	(wire
-		(pts
 			(xy 297.18 133.35) (xy 334.01 133.35)
 		)
@@
 	(wire
 		(pts
+			(xy 241.3 74.93) (xy 241.3 86.36)
+		)
+		(stroke
+			(width 0)
+			(type default)
+		)
+	)
+	(wire
+		(pts
 			(xy 241.3 86.36) (xy 257.81 86.36)
 		)
@@
 	(wire
 		(pts
-			(xy 241.3 68.58) (xy 241.3 57.15)
-		)
-		(stroke
-			(width 0)
-			(type default)
-		)
-	)
-	(wire
-		(pts
 			(xy 222.25 120.65) (xy 223.52 120.65)
 		)
@@
 	(wire
 		(pts
+			(xy 241.3 57.15) (xy 241.3 69.85)
+		)
+		(stroke
+			(width 0)
+			(type default)
+		)
+	)
+	(wire
+		(pts
 			(xy 327.66 86.36) (xy 320.04 86.36)
 		)
@@
 	(wire
 		(pts
-			(xy 241.3 76.2) (xy 241.3 86.36)
-		)
-		(stroke
-			(width 0)
-			(type default)
-		)
-	)
-	(wire
-		(pts
 			(xy 223.52 20.32) (xy 257.81 20.32)
 		)
@@
 	(wire
 		(pts
+			(xy 146.05 63.5) (xy 146.05 66.04)
+		)
+		(stroke
+			(width 0)
+			(type default)
+		)
+	)
+	(wire
+		(pts
 			(xy 146.05 66.04) (xy 146.05 68.58)
 		)
@@
 		)
 	)
-	(label "LED_INFO_BIO_12V"
-		(at 133.35 63.5 180)
-		(effects
-			(font
-				(size 1.27 1.27)
-			)
-			(justify right bottom)
+	(label "LED_INFO_REC_12V"
+		(at 146.05 60.96 0)
+		(effects
+			(font
+				(size 1.27 1.27)
+			)
+			(justify left bottom)
 		)
 	)
@@
 		)
 	)
-	(label "LED_INFO_REC_12V"
-		(at 146.05 63.5 0)
-		(effects
-			(font
-				(size 1.27 1.27)
-			)
-			(justify left bottom)
-		)
-	)
 	(label "GND"
 		(at 238.76 118.11 0)
@@
 		)
 	)
-	(label "LED_INFO_OPEN_12V"
-		(at 133.35 66.04 180)
+	(label "LED_INFO_BIO_12V"
+		(at 133.35 60.96 180)
 		(effects
 			(font
@@
 			)
 			(justify left bottom)
+		)
+	)
+	(label "LED_INFO_OPEN_12V"
+		(at 133.35 63.5 180)
+		(effects
+			(font
+				(size 1.27 1.27)
+			)
+			(justify right bottom)
 		)
 	)
@@
 	)
 	(symbol
-		(lib_id "Device:C_Polarized")
+		(lib_id "Device:C_Small")
 		(at 241.3 72.39 0)
 		(unit 1)
@@
 		(fields_autoplaced yes)
 		(property "Reference" "C51"
-			(at 245.11 70.2309 0)
+			(at 243.84 71.1262 0)
 			(effects
 				(font
@@
 		)
 		(property "Value" "0.1 µF"
-			(at 245.11 72.7709 0)
+			(at 243.84 73.6662 0)
 			(effects
 				(font
@@
 		)
 		(property "Footprint" "C_0603_1608Metric"
-			(at 242.2652 76.2 0)
+			(at 241.3 72.39 0)
 			(effects
 				(font
@@
 			)
 		)
-		(property "Description" "Polarized capacitor"
+		(property "Description" "Unpolarized capacitor, small symbol"
 			(at 241.3 72.39 0)
 			(effects
@@
 	)
 	(symbol
-		(lib_id "Connector_Generic:Conn_02x03_Odd_Even")
+		(lib_id "Connector_Generic:Conn_02x05_Odd_Even")
 		(at 138.43 66.04 0)
 		(unit 1)
@@
 		(fields_autoplaced yes)
 		(property "Reference" "J15"
+			(at 139.7 54.61 0)
+			(effects
+				(font
+					(size 1.27 1.27)
+				)
+			)
+		)
+		(property "Value" "IDC-10_ZONE_INFO_12V"
 			(at 139.7 57.15 0)
 			(effects
@@
 			)
 		)
-		(property "Value" "IDC-6_ZONE_INFO_12V"
-			(at 139.7 59.69 0)
-			(effects
-				(font
-					(size 1.27 1.27)
-				)
-			)
-		)
-		(property "Footprint" "Connector_IDC:IDC-Header_2x03_P2.54mm_Vertical"
+		(property "Footprint" "Connector_IDC:IDC-Header_2x05_P2.54mm_Vertical"
 			(at 138.43 66.04 0)
 			(effects
@@
 			)
 		)
-		(property "Description" "Generic connector, double row, 02x03, odd/even pin numbering scheme (row 1 odd numbers, row 2 even numbers), script generated (kicad-library-utils/schlib/autogen/connector/)"
+		(property "Description" "Generic connector, double row, 02x05, odd/even pin numbering scheme (row 1 odd numbers, row 2 even numbers), script generated (kicad-library-utils/schlib/autogen/connector/)"
 			(at 138.43 66.04 0)
 			(effects
@@
 		(pin "6"
 		)
+		(pin "9"
+		)
+		(pin "8"
+		)
+		(pin "10"
+		)
+		(pin "7"
+		)
 		(instances
