File: hardware/pcb/powerplant.kicad_sch (KiCad schematic)
At the start: 91 parts, among them J16 14_NIXIE_BUS, J17 J_AUDIO_OUT, J18 J_MIC, J19 J_LIGHT, J21 IDC-10_METER_SIG, J22 J_IN, J23 J_OUT, J24 POWER IN 12V, J6 RPi_GPIO, Q1 IRLZ44N, Q2 IRLZ44N, Q3 IRLZ44N, Q4 IRLZ44N, Q5 IRLZ44N, Q6 IRLZ44N, U1 MCP4728, U10 LM358_DFN, U14 PCM5102A, U2 LM358_DFN, U3 LM358_DFN, U4 MCP4728

Commit message: Update hardware schematics and documentation; added source of truth for hardware, removed unused symbols, and modified connector specifications.
Parts:
- removed C29, C56: 100 nF, Capacitor_SMD:C_0603_1608Metric, symbol Device:C
- removed C55: 10 µF, Capacitor_SMD:C_1206_3216Metric_Pad1.33x1.80mm_HandSolder, symbol Device:C_Polarized
- removed C57: 1 µF, C_0603_1608Metric, symbol Device:C
- removed FB1: FerriteBead 600 Ω @ 100 MHz, Inductor_SMD:L_1206_3216Metric_Pad1.22x1.90mm_HandSolder, symbol Device:FerriteBead
- removed J17: J_AUDIO_OUT, Connector_Phoenix_MSTB:PhoenixContact_MSTBVA_2,5_3-G-5,08_1x03_P5.08mm_Vertical, symbol Connector:Conn_01x03_Socket
- removed J18: J_MIC, Connector_JST:JST_PH_B6B-PH-K_1x06_P2.00mm_Vertical, symbol Connector:Conn_01x06_Pin
- removed R31, R32, R61: 33 Ω, Resistor_SMD:R_0603_1608Metric, symbol Device:R
- removed U14: PCM5102A, Package_SO:TSSOP-20_4.4x6.5mm_P0.65mm, symbol Audio:PCM5102A
- added A1: RaspberryPi_Pico, Module:RaspberryPi_Pico_Common_Unspecified, symbol MCU_Module:RaspberryPi_Pico
- added C29: 10 µF, Resistor_SMD:R_1206_3216Metric, symbol Device:C_Polarized
- added J2: J_AUX, Connector_JST:JST_PH_B8B-PH-K_1x08_P2.00mm_Vertical, symbol Connector:Conn_01x08_Pin
- added J3: VL53L0X, Connector_JST:JST_PH_B4B-PH-K_1x04_P2.00mm_Vertical, symbol Connector_Generic:Conn_01x04
- added J4: J_LCD_PWR, Connector_JST:JST_PH_B2B-PH-K_1x02_P2.00mm_Vertical, symbol Connector_Generic:Conn_01x02
- added J5: SPARE, Connector_JST:JST_PH_B8B-PH-K_1x08_P2.00mm_Vertical, symbol Connector_Generic:Conn_01x08
- added U14: TPS22917DBV, Package_TO_SOT_SMD:SOT-23-6, symbol Power_Management:TPS22917DBV
- C1, C11, C13, C18, C20, C4, C8: footprint Capacitor_SMD:C_1206_3216Metric_Pad1.33x1.80mm_HandSolder -> Resistor_SMD:R_1206_3216Metric
- C53: value 100 nF -> 1 µF
- C54: value 100 nF -> 4.7 µF
Connections:
- net +12V: now also C29.1
- net +3.3V: now also J5.1 (Pin_1)
- net +5V: now also C53.2, A1.40 (VBUS), J3.4 (Pin_4), U14.1 (VIN); no longer C53.1, C54.2
- net GND: now also C53.1, C54.2, J23.2 (Pin_2), NT1.1, A1.13 (GND), A1.18 (GND), A1.23 (GND), A1.28 (GND), A1.3 (GND), A1.38 (GND), A1.8 (GND), J2.7 (Pin_7), J3.1 (Pin_1), J4.2 (Pin_2), J5.2 (Pin_2), U14.2 (GND); no longer C1.2, C10.1, C11.2, C12.1, C13.2, C17.1, C18.2, C19.1, C2.1, C20.2, C53.2, C54.1, C7.1, C8.2, NT1.2, R13.2, R14.2, R17.1, R18.1, R19.1, R20.1, R25.1, R26.1, R27.2, R28.2, R4.2, R8.2
- net GNDPWR: now also C1.2, C10.1, C11.2, C12.1, C13.2, C17.1, C18.2, C19.1, C2.1, C20.2, C7.1, C8.2, NT1.2, R13.2, R14.2, R17.1, R18.1, R19.1, R20.1, R25.1, R26.1, R27.2, R28.2, R4.2, R8.2, C29.2; no longer J23.2 (Pin_2), NT1.1
- net GPIO_LED1: no longer names the net of J6.7 (BCM4_GPCLK0)
- net GPIO_LED2: no longer names the net of J6.29 (BCM5)
- net GPIO_LED3: no longer names the net of J6.31 (BCM6)
- net GPIO_LED4 renamed GP1_RX_PICO
- net GP1_RX_PICO: now also A1.2 (GPIO1)
- net GPIO_LED5 renamed GP0_TX_PICO
- net GP0_TX_PICO: now also A1.1 (GPIO0)
- net GPIO_VOL_RING: no longer names the net of J6.37 (BCM26)
- net I2C_SCL renamed AUX_SCL
- net AUX_SCL: now also J2.6 (Pin_6), J3.2 (Pin_2)
- net I2C_SDA renamed AUX_SDA
- net AUX_SDA: now also J2.5 (Pin_5), J3.3 (Pin_3)
- net I2S_BCK renamed LCD_PWR_EN
- net LCD_PWR_EN: now also U14.3 (ON)
- net I2S_DIN renamed AUX_I2S_TX
- net AUX_I2S_TX: now also J2.3 (Pin_3)
- net I2S_LRCK renamed AUX_I2S_LRCLK
- net AUX_I2S_LRCLK: now also J2.2 (Pin_2)
- net LED_MODE_DATA_IN: no longer names the net of J6.33 (BCM13_PWM1)
- net LED_RANGE_DATA_IN: no longer names the net of J6.32 (BCM12_PWM0)
- net LED_TEMP_DATA_IN: no longer names the net of J6.36 (BCM16)
- net MIC_I2S_DOUT renamed AUX_I2S_RX
- net AUX_I2S_RX: now also J2.4 (Pin_4)
- new net: C54.1, J4.1 (Pin_1), U14.6 (VOUT)
- new net BLK_METER_LED/GPIO_LED1: A1.9 (GPIO6)
- new net BLK_METER_LED/GPIO_LED2: A1.10 (GPIO7)
- new net BLK_METER_LED/GPIO_LED3: A1.11 (GPIO8)
- new net BLK_METER_LED/GPIO_LED4: A1.12 (GPIO9)
- new net BLK_METER_LED/GPIO_LED5: A1.14 (GPIO10)
- new net BLK_METER_LED/GPIO_VOL_RING: A1.7 (GPIO5)
- new net BLK_SWITCH_LED/LED_MODE_DATA_IN: A1.5 (GPIO3)
- new net BLK_SWITCH_LED/LED_RANGE_DATA_IN: A1.4 (GPIO2)
- new net BLK_SWITCH_LED/LED_TEMP_DATA_IN: A1.6 (GPIO4)
- new net GP11: A1.15 (GPIO11), J5.3 (Pin_3)
- new net GP12: A1.16 (GPIO12), J5.4 (Pin_4)
- new net GP13: A1.17 (GPIO13), J5.5 (Pin_5)
- new net GP14: A1.19 (GPIO14), J5.6 (Pin_6)
- new net GP15: A1.20 (GPIO15), J5.7 (Pin_7)
- new net GP16: A1.21 (GPIO16), J5.8 (Pin_8)
- no-connect marks 27 -> 23
Other:
- note removed: "AUDIO, WYJSCIE NA WZMACNIACZ/GLOSNIKI"
- note removed: "WEJSCIE MIC"
- moved on the sheet: C58, C59, C61, FB2, J19, J23, NT1, U10C
